Commit message: display_head.launch.py shows stl files for head

File: src/hros5_description/urdf/minimal.urdf.xacro (robot description, xacro)
@@ -2,5 +2,5 @@
 <robot xmlns:xacro="http://ros.org/wiki/xacro" name="test_bot">
   <xacro:include filename="torso/torso.xacro"/>
-  <xacro:include filename="head/head_debug.xacro"/>
+  <xacro:include filename="head/head.xacro"/>
   <xacro:include filename="arms/left_arm_debug.xacro"/>
   <xacro:include filename="arms/right_arm_debug.xacro"/>

File: src/hros5_description/urdf/torso/torso.xacro (robot description, xacro)
@@ -12,5 +12,5 @@
       <origin xyz="0 0 0" rpy="0 0 0"/>
       <geometry>
-        <mesh filename="package://hros5_description/meshes/torso/torso.stl" scale="1 1 1"/>
+        <mesh filename="package://hros5_description/meshes/torso/torso.stl" scale="0.1 0.1 0.1"/>
       </geometry>
     </visual>
@@ -18,5 +18,5 @@
       <origin xyz="0 0 0" rpy="0 0 0"/>
       <geometry>
-        <mesh filename="package://hros5_description/meshes/torso/torso.stl" scale="1 1 1"/>
+        <mesh filename="package://hros5_description/meshes/torso/torso.stl" scale="0.1 0.1 0.1"/>
       </geometry>
     </collision>
