Commit message: Changed hw interface and moved ros2_control to hros5_control

File: src/hros5_description/urdf/hros5.xacro (robot description, xacro)
@@ -2,5 +2,5 @@
 <robot name="hros5" xmlns:xacro="http://www.ros.org/wiki/xacro">
 	<xacro:include filename="$(find hros5_description)/urdf/hros5_control.xacro" />
-	<xacro:include filename="$(find hros5_description)/urdf/hros5_gazebo.xacro" />
+	<!--xacro:include filename="$(find hros5_description)/urdf/hros5_gazebo.xacro" /-->
 	<xacro:include filename="$(find hros5_description)/urdf/robot/robot.xacro" />
 </robot>

File: src/hros5_description/urdf/hros5_control.xacro (robot description, xacro)
@@ -7,8 +7,8 @@
 			<type>transmission_interface/SimpleTransmission</type>
 			<joint name="HeadYaw">
-				<hardwareInterface>EffortJointInterface</hardwareInterface>
+				<hardwareInterface>hardware_interface/PositionJointInterface</hardwareInterface>
 			</joint>
 			<actuator name="HeadYaw_Motor">
-				<hardwareInterface>EffortJointInterface</hardwareInterface>
+				<hardwareInterface>hardware_interface/PositionJointInterface</hardwareInterface>
 				<mechanicalReduction>1</mechanicalReduction>
 			</actuator>
@@ -17,8 +17,8 @@
 			<type>transmission_interface/SimpleTransmission</type>
 			<joint name="HeadPitch">
-				<hardwareInterface>EffortJointInterface</hardwareInterface>
+				<hardwareInterface>hardware_interface/PositionJointInterface</hardwareInterface>
 			</joint>
 			<actuator name="HeadPitch_Motor">
-				<hardwareInterface>EffortJointInterface</hardwareInterface>
+				<hardwareInterface>hardware_interface/PositionJointInterface</hardwareInterface>
 				<mechanicalReduction>1</mechanicalReduction>
 			</actuator>
@@ -32,8 +32,8 @@
 			<type>transmission_interface/SimpleTransmission</type>
 			<joint name="${side}ShoulderPitch">
-				<hardwareInterface>EffortJointInterface</hardwareInterface>
+				<hardwareInterface>hardware_interface/PositionJointInterface</hardwareInterface>
 			</joint>
 			<actuator name="${side}ShoulderPitch_Motor">
-				<hardwareInterface>EffortJointInterface</hardwareInterface>
+				<hardwareInterface>hardware_interface/PositionJointInterface</hardwareInterface>
 				<mechanicalReduction>1</mechanicalReduction>
 			</actuator>
@@ -42,8 +42,8 @@
 			<type>transmission_interface/SimpleTransmission</type>
 			<joint name="${side}ShoulderRoll">
-				<hardwareInterface>EffortJointInterface</hardwareInterface>
+				<hardwareInterface>hardware_interface/PositionJointInterface</hardwareInterface>
 			</joint>
 			<actuator name="${side}ShoulderRoll_Motor">
-				<hardwareInterface>EffortJointInterface</hardwareInterface>
+				<hardwareInterface>hardware_interface/PositionJointInterface</hardwareInterface>
 				<mechanicalReduction>1</mechanicalReduction>
 			</actuator>
@@ -52,8 +52,8 @@
 			<type>transmission_interface/SimpleTransmission</type>
 			<joint name="${side}ElbowPitch">
-				<hardwareInterface>EffortJointInterface</hardwareInterface>
+				<hardwareInterface>hardware_interface/PositionJointInterface</hardwareInterface>
 			</joint>
 			<actuator name="${side}ElbowPitch_Motor">
-				<hardwareInterface>EffortJointInterface</hardwareInterface>
+				<hardwareInterface>hardware_interface/PositionJointInterface</hardwareInterface>
 				<mechanicalReduction>1</mechanicalReduction>
 			</actuator>
@@ -68,8 +68,8 @@
 			<type>transmission_interface/SimpleTransmission</type>
 			<joint name="${side}HipYaw">
-				<hardwareInterface>EffortJointInterface</hardwareInterface>
+				<hardwareInterface>hardware_interface/PositionJointInterface</hardwareInterface>
 			</joint>
 			<actuator name="${side}HipYaw_Motor">
-				<hardwareInterface>EffortJointInterface</hardwareInterface>
+				<hardwareInterface>hardware_interface/PositionJointInterface</hardwareInterface>
 				<mechanicalReduction>1</mechanicalReduction>
 			</actuator>
@@ -78,8 +78,8 @@
 			<type>transmission_interface/SimpleTransmission</type>
 			<joint name="${side}HipRoll">
-				<hardwareInterface>EffortJointInterface</hardwareInterface>
+				<hardwareInterface>hardware_interface/PositionJointInterface</hardwareInterface>
 			</joint>
 			<actuator name="${side}HipRoll_Motor">
-				<hardwareInterface>EffortJointInterface</hardwareInterface>
+				<hardwareInterface>hardware_interface/PositionJointInterface</hardwareInterface>
 				<mechanicalReduction>1</mechanicalReduction>
 			</actuator>
@@ -88,8 +88,8 @@
 			<type>transmission_interface/SimpleTransmission</type>
 			<joint name="${side}HipPitch">
-				<hardwareInterface>EffortJointInterface</hardwareInterface>
+				<hardwareInterface>hardware_interface/PositionJointInterface</hardwareInterface>
 			</joint>
 			<actuator name="${side}HipPitch_Motor">
-				<hardwareInterface>EffortJointInterface</hardwareInterface>
+				<hardwareInterface>hardware_interface/PositionJointInterface</hardwareInterface>
 				<mechanicalReduction>1</mechanicalReduction>
 			</actuator>
@@ -98,8 +98,8 @@
 			<type>transmission_interface/SimpleTransmission</type>
 			<joint name="${side}KneePitch">
-				<hardwareInterface>EffortJointInterface</hardwareInterface>
+				<hardwareInterface>hardware_interface/PositionJointInterface</hardwareInterface>
 			</joint>
 			<actuator name="${side}KneePitch_Motor">
-				<hardwareInterface>EffortJointInterface</hardwareInterface>
+				<hardwareInterface>hardware_interface/PositionJointInterface</hardwareInterface>
 				<mechanicalReduction>1</mechanicalReduction>
 			</actuator>
@@ -108,8 +108,8 @@
 			<type>transmission_interface/SimpleTransmission</type>
 			<joint name="${side}AnklePitch">
-				<hardwareInterface>EffortJointInterface</hardwareInterface>
+				<hardwareInterface>hardware_interface/PositionJointInterface</hardwareInterface>
 			</joint>
 			<actuator name="${side}AnklePitch_Motor">
-				<hardwareInterface>EffortJointInterface</hardwareInterface>
+				<hardwareInterface>hardware_interface/PositionJointInterface</hardwareInterface>
 				<mechanicalReduction>1</mechanicalReduction>
 			</actuator>
@@ -118,8 +118,8 @@
 			<type>transmission_interface/SimpleTransmission</type>
 			<joint name="${side}AnkleRoll">
-				<hardwareInterface>EffortJointInterface</hardwareInterface>
+				<hardwareInterface>hardware_interface/PositionJointInterface</hardwareInterface>
 			</joint>
 			<actuator name="${side}AnkleRoll_Motor">
-				<hardwareInterface>EffortJointInterface</hardwareInterface>
+				<hardwareInterface>hardware_interface/PositionJointInterface</hardwareInterface>
 				<mechanicalReduction>1</mechanicalReduction>
 			</actuator>
@@ -128,3 +128,57 @@
 	<xacro:leg_joints_transmissions side="L"/>
 	<xacro:leg_joints_transmissions side="R"/>
+	<!-- ROS 2 Control System Configuration -->
+	<ros2_control name="DynamixelHardware" type="system">
+	  <hardware>
+		<plugin>dynamixel_hardware/DynamixelHardware</plugin>
+	  </hardware>
+	  <joint name="LHipYaw">
+		<command_interface name="position"/>
+		<state_interface name="position"/>
+	  </joint>
+	  <joint name="LHipRoll">
+		<command_interface name="position"/>
+		<state_interface name="position"/>
+	  </joint>
+	  <joint name="LHipPitch">
+		<command_interface name="position"/>
+		<state_interface name="position"/>
+	  </joint>
+	  <joint name="LKneePitch">
+		<command_interface name="position"/>
+		<state_interface name="position"/>
+	  </joint>
+	  <joint name="LAnklePitch">
+		<command_interface name="position"/>
+		<state_interface name="position"/>
+	  </joint>
+	  <joint name="LAnkleRoll">
+		<command_interface name="position"/>
+		<state_interface name="position"/>
+	  </joint>
+	  <joint name="RHipYaw">
+		<command_interface name="position"/>
+		<state_interface name="position"/>
+	  </joint>
+	  <joint name="RHipRoll">
+		<command_interface name="position"/>
+		<state_interface name="position"/>
+	  </joint>
+	  <joint name="RHipPitch">
+		<command_interface name="position"/>
+		<state_interface name="position"/>
+	  </joint>
+	  <joint name="RKneePitch">
+		<command_interface name="position"/>
+		<state_interface name="position"/>
+	  </joint>
+	  <joint name="RAnklePitch">
+		<command_interface name="position"/>
+		<state_interface name="position"/>
+	  </joint>
+	  <joint name="RAnkleRoll">
+		<command_interface name="position"/>
+		<state_interface name="position"/>
+	  </joint>
+	</ros2_control>
 </robot>

File: src/hros5_description/urdf/legs/legs.xacro (robot description, xacro)
@@ -120,232 +120,3 @@
 	</joint>
 	<link name="r_sole"/>
-  <ros2_control name="HROS5DynamixelSystem" type="system">
-    <hardware>
-      <plugin>ros2_control_dynamixel_hardware/DynamixelSystemHardware</plugin>
-    </hardware>
-    <!-- Each joint used in the legs should have a control interface -->
-    <joint name="left_hip_yaw">
-      <command_interface name="position"/>
-      <state_interface name="position"/>
-      <state_interface name="velocity"/>
-    </joint>
-    <joint name="left_hip_roll">
-      <command_interface name="position"/>
-      <state_interface name="position"/>
-      <state_interface name="velocity"/>
-    </joint>
-    <joint name="left_hip_pitch">
-      <command_interface name="position"/>
-      <state_interface name="position"/>
-      <state_interface name="velocity"/>
-    </joint>
-    <joint name="left_knee">
-      <command_interface name="position"/>
-      <state_interface name="position"/>
-      <state_interface name="velocity"/>
-    </joint>
-    <joint name="left_ankle_pitch">
-      <command_interface name="position"/>
-      <state_interface name="position"/>
-      <state_interface name="velocity"/>
-    </joint>
-    <joint name="left_ankle_roll">
-      <command_interface name="position"/>
-      <state_interface name="position"/>
-      <state_interface name="velocity"/>
-    </joint>
-    <joint name="right_hip_yaw">
-      <command_interface name="position"/>
-      <state_interface name="position"/>
-      <state_interface name="velocity"/>
-    </joint>
-    <joint name="right_hip_roll">
-      <command_interface name="position"/>
-      <state_interface name="position"/>
-      <state_interface name="velocity"/>
-    </joint>
-    <joint name="right_hip_pitch">
-      <command_interface name="position"/>
-      <state_interface name="position"/>
-      <state_interface name="velocity"/>
-    </joint>
-    <joint name="right_knee">
-      <command_interface name="position"/>
-      <state_interface name="position"/>
-      <state_interface name="velocity"/>
-    </joint>
-    <joint name="right_ankle_pitch">
-      <command_interface name="position"/>
-      <state_interface name="position"/>
-      <state_interface name="velocity"/>
-    </joint>
-    <joint name="right_ankle_roll">
-      <command_interface name="position"/>
-      <state_interface name="position"/>
-      <state_interface name="velocity"/>
-    </joint>
-  </ros2_control>
-  <ros2_control name="DynamixelHardware" type="system">
-    <hardware>
-      <plugin>ros2_control_dynamixel/DynamixelSystemHardware</plugin>
-    </hardware>
-    <!-- LEFT LEG -->
-    <joint name="left_hip_yaw">
-      <command_interface name="position"/>
-      <state_interface name="position"/>
-    </joint>
-    <joint name="left_hip_roll">
-      <command_interface name="position"/>
-      <state_interface name="position"/>
-    </joint>
-    <joint name="left_hip_pitch">
-      <command_interface name="position"/>
-      <state_interface name="position"/>
-    </joint>
-    <joint name="left_knee">
-      <command_interface name="position"/>
-      <state_interface name="position"/>
-    </joint>
-    <joint name="left_ankle_pitch">
-      <command_interface name="position"/>
-      <state_interface name="position"/>
-    </joint>
-    <joint name="left_ankle_roll">
-      <command_interface name="position"/>
-      <state_interface name="position"/>
-    </joint>
-    <!-- RIGHT LEG -->
-    <joint name="right_hip_yaw">
-      <command_interface name="position"/>
-      <state_interface name="position"/>
-    </joint>
-    <joint name="right_hip_roll">
-      <command_interface name="position"/>
-      <state_interface name="position"/>
-    </joint>
-    <joint name="right_hip_pitch">
-      <command_interface name="position"/>
-      <state_interface name="position"/>
-    </joint>
-    <joint name="right_knee">
-      <command_interface name="position"/>
-      <state_interface name="position"/>
-    </joint>
-    <joint name="right_ankle_pitch">
-      <command_interface name="position"/>
-      <state_interface name="position"/>
-    </joint>
-    <joint name="right_ankle_roll">
-      <command_interface name="position"/>
-      <state_interface name="position"/>
-    </joint>
-  </ros2_control>
-  <transmission name="left_hip_yaw_trans">
-    <type>transmission_interface/SimpleTransmission</type>
-    <joint name="left_hip_yaw">
-      <hardwareInterface>hardware_interface/PositionJointInterface</hardwareInterface>
-    </joint>
-    <actuator name="left_hip_yaw_motor">
-      <hardwareInterface>hardware_interface/PositionJointInterface</hardwareInterface>
-    </actuator>
-  </transmission>
-  <transmission name="left_hip_roll_trans">
-    <type>transmission_interface/SimpleTransmission</type>
-    <joint name="left_hip_roll">
-      <hardwareInterface>hardware_interface/PositionJointInterface</hardwareInterface>
-    </joint>
-    <actuator name="left_hip_roll_motor">
-      <hardwareInterface>hardware_interface/PositionJointInterface</hardwareInterface>
-    </actuator>
-  </transmission>
-  <transmission name="left_hip_pitch_trans">
-    <type>transmission_interface/SimpleTransmission</type>
-    <joint name="left_hip_pitch">
-      <hardwareInterface>hardware_interface/PositionJointInterface</hardwareInterface>
-    </joint>
-    <actuator name="left_hip_pitch_motor">
-      <hardwareInterface>hardware_interface/PositionJointInterface</hardwareInterface>
-    </actuator>
-  </transmission>
-  <transmission name="left_knee_trans">
-    <type>transmission_interface/SimpleTransmission</type>
-    <joint name="left_knee">
-      <hardwareInterface>hardware_interface/PositionJointInterface</hardwareInterface>
-    </joint>
-    <actuator name="left_knee_motor">
-      <hardwareInterface>hardware_interface/PositionJointInterface</hardwareInterface>
-    </actuator>
-  </transmission>
-  <transmission name="left_ankle_pitch_trans">
-    <type>transmission_interface/SimpleTransmission</type>
-    <joint name="left_ankle_pitch">
-      <hardwareInterface>hardware_interface/PositionJointInterface</hardwareInterface>
-    </joint>
-    <actuator name="left_ankle_pitch_motor">
-      <hardwareInterface>hardware_interface/PositionJointInterface</hardwareInterface>
-    </actuator>
-  </transmission>
-  <transmission name="left_ankle_roll_trans">
-    <type>transmission_interface/SimpleTransmission</type>
-    <joint name="left_ankle_roll">
-      <hardwareInterface>hardware_interface/PositionJointInterface</hardwareInterface>
-    </joint>
-    <actuator name="left_ankle_roll_motor">
-      <hardwareInterface>hardware_interface/PositionJointInterface</hardwareInterface>
-    </actuator>
-  </transmission>
-  <transmission name="right_hip_yaw_trans">
-    <type>transmission_interface/SimpleTransmission</type>
-    <joint name="right_hip_yaw">
-      <hardwareInterface>hardware_interface/PositionJointInterface</hardwareInterface>
-    </joint>
-    <actuator name="right_hip_yaw_motor">
-      <hardwareInterface>hardware_interface/PositionJointInterface</hardwareInterface>
-    </actuator>
-  </transmission>
-  <transmission name="right_hip_roll_trans">
-    <type>transmission_interface/SimpleTransmission</type>
-    <joint name="right_hip_roll">
-      <hardwareInterface>hardware_interface/PositionJointInterface</hardwareInterface>
-    </joint>
-    <actuator name="right_hip_roll_motor">
-      <hardwareInterface>hardware_interface/PositionJointInterface</hardwareInterface>
-    </actuator>
-  </transmission>
-  <transmission name="right_hip_pitch_trans">
-    <type>transmission_interface/SimpleTransmission</type>
-    <joint name="right_hip_pitch">
-      <hardwareInterface>hardware_interface/PositionJointInterface</hardwareInterface>
-    </joint>
-    <actuator name="right_hip_pitch_motor">
-      <hardwareInterface>hardware_interface/PositionJointInterface</hardwareInterface>
-    </actuator>
-  </transmission>
-  <transmission name="right_knee_trans">
-    <type>transmission_interface/SimpleTransmission</type>
-    <joint name="right_knee">
-      <hardwareInterface>hardware_interface/PositionJointInterface</hardwareInterface>
-    </joint>
-    <actuator name="right_knee_motor">
-      <hardwareInterface>hardware_interface/PositionJointInterface</hardwareInterface>
-    </actuator>
-  </transmission>
-  <transmission name="right_ankle_pitch_trans">
-    <type>transmission_interface/SimpleTransmission</type>
-    <joint name="right_ankle_pitch">
-      <hardwareInterface>hardware_interface/PositionJointInterface</hardwareInterface>
-    </joint>
-    <actuator name="right_ankle_pitch_motor">
-      <hardwareInterface>hardware_interface/PositionJointInterface</hardwareInterface>
-    </actuator>
-  </transmission>
-  <transmission name="right_ankle_roll_trans">
-    <type>transmission_interface/SimpleTransmission</type>
-    <joint name="right_ankle_roll">
-      <hardwareInterface>hardware_interface/PositionJointInterface</hardwareInterface>
-    </joint>
-    <actuator name="right_ankle_roll_motor">
-      <hardwareInterface>hardware_interface/PositionJointInterface</hardwareInterface>
-    </actuator>
-  </transmission>
 </robot>
