Commit message: Fixed typo

File: src/hros5_description/urdf/hros5_control.xacro (robot description, xacro)
@@ -3,5 +3,5 @@
 <!-- HEAD -->
 	<!-- XACRO -->
-	<xacro:macro name="head_trasmissions">
+	<xacro:macro name="head_transmissions">
 		<transmission name="HeadYaw_Transmission">
 			<type>transmission_interface/SimpleTransmission</type>
@@ -25,5 +25,5 @@
 		</transmission>
 	</xacro:macro>
-	<xacro:head_trasmissions/>
+	<xacro:head_transmissions/>
 <!-- ARMS -->
 	<!-- XACRO -->
