Commit message: Working RViz setup with modular robot.xacro includes

File: src/hros5_description/urdf/hros5_visuals_collisions_endoskeleton.xacro (robot description, xacro)
@@ -6,5 +6,5 @@
 			<origin xyz="0 0 0" rpy="0 0 0"/>
 			<geometry>
-				<mesh filename="package://hros5_description/meshes/endoskeleton/visual/torso.dae" scale="${scale} ${scale} ${scale}"/>
+				<mesh filename="package://hros5_description/meshes/torso/torso.dae" scale="${scale} ${scale} ${scale}"/>
 			</geometry>
 		</visual>
@@ -12,5 +12,5 @@
 			<origin xyz="0 0 0" rpy="0 0 0"/>
 			<geometry>
-				<mesh filename="package://hros5_description/meshes/endoskeleton/collision/torso.stl" scale="${scale} ${scale} ${scale}"/>
+				<mesh filename="package://hros5_description/meshes/torso/torso.stl" scale="${scale} ${scale} ${scale}"/>
 			</geometry>
 		</collision>
@@ -22,5 +22,5 @@
 			<origin xyz="-0.03 0 0.033" rpy="0 0 0"/>
 			<geometry>
-				<mesh filename="package://hros5_description/meshes/endoskeleton/visual/LowerHead.dae" scale="${scale} ${scale} ${scale}"/>
+				<mesh filename="package://hros5_description/meshes/head/LowerHead.dae" scale="${scale} ${scale} ${scale}"/>
 			</geometry>
 		</visual>
@@ -28,5 +28,5 @@
 			<origin xyz="-0.03 0 0.033" rpy="0 0 0"/>
 			<geometry>
-				<mesh filename="package://hros5_description/meshes/endoskeleton/collision/LowerHead.stl" scale="${scale} ${scale} ${scale}"/>
+				<mesh filename="package://hros5_description/meshes/head/LowerHead.stl" scale="${scale} ${scale} ${scale}"/>
 			</geometry>
 		</collision>
@@ -37,5 +37,5 @@
 			<origin xyz="0.0075 -0.0045 0.0275" rpy="0 0 0"/>
 			<geometry>
-				<mesh filename="package://hros5_description/meshes/endoskeleton/visual/UpperHeadBase.dae" scale="${scale} ${scale} ${scale}"/>
+				<mesh filename="package://hros5_description/meshes/head/UpperHeadBase.dae" scale="${scale} ${scale} ${scale}"/>
 			</geometry>
 		</visual>
@@ -43,5 +43,5 @@
 			<origin xyz="0.0075 -0.0045 0.0275" rpy="0 0 0"/>
 			<geometry>
-				<mesh filename="package://hros5_description/meshes/endoskeleton/collision/UpperHeadBase.stl" scale="${scale} ${scale} ${scale}"/>
+				<mesh filename="package://hros5_description/meshes/head/UpperHeadBase.stl" scale="${scale} ${scale} ${scale}"/>
 			</geometry>
 		</collision>
@@ -51,5 +51,5 @@
 			<origin xyz="-0.03 0 0.00075" rpy="0 0 0"/>
 			<geometry>
-				<mesh filename="package://hros5_description/meshes/endoskeleton/visual/UpperHeadMotor.dae" scale="${scale} ${scale} ${scale}"/>
+				<mesh filename="package://hros5_description/meshes/head/UpperHeadMotor.dae" scale="${scale} ${scale} ${scale}"/>
 			</geometry>
 		</visual>
@@ -57,5 +57,5 @@
 			<origin xyz="-0.03 0 0.00075" rpy="0 0 0"/>
 			<geometry>
-				<mesh filename="package://hros5_description/meshes/endoskeleton/collision/UpperHeadMotor.stl" scale="${scale} ${scale} ${scale}"/>
+				<mesh filename="package://hros5_description/meshes/head/UpperHeadMotor.stl" scale="${scale} ${scale} ${scale}"/>
 			</geometry>
 		</collision>
@@ -65,5 +65,5 @@
 			<origin xyz="0.001 0 0.0375" rpy="0 0 0"/>
 			<geometry>
-				<mesh filename="package://hros5_description/meshes/endoskeleton/visual/UpperHeadBack.dae" scale="${scale} ${scale} ${scale}"/>
+				<mesh filename="package://hros5_description/meshes/head/UpperHeadBack.dae" scale="${scale} ${scale} ${scale}"/>
 			</geometry>
 		</visual>
@@ -71,5 +71,5 @@
 			<origin xyz="0.001 0 0.0375" rpy="0 0 0"/>
 			<geometry>
-				<mesh filename="package://hros5_description/meshes/endoskeleton/collision/UpperHeadBack.stl" scale="${scale} ${scale} ${scale}"/>
+				<mesh filename="package://hros5_description/meshes/head/UpperHeadBack.stl" scale="${scale} ${scale} ${scale}"/>
 			</geometry>
 		</collision>
@@ -81,5 +81,5 @@
 			<origin xyz="0 ${reflect*0.0122} -0.0125" rpy="0 0 0"/>
 			<geometry>
-				<mesh filename="package://hros5_description/meshes/endoskeleton/visual/${side}Shoulder.dae" scale="${scale} ${scale} ${scale}"/>
+				<mesh filename="package://hros5_description/meshes/arms/${side}Shoulder.dae" scale="${scale} ${scale} ${scale}"/>
 			</geometry>
 		</visual>
@@ -87,5 +87,5 @@
 			<origin xyz="0 ${reflect*0.0122} -0.0125" rpy="0 0 0"/>
 			<geometry>
-				<mesh filename="package://hros5_description/meshes/endoskeleton/collision/${side}Shoulder.stl" scale="${scale} ${scale} ${scale}"/>
+				<mesh filename="package://hros5_description/meshes/arms/${side}Shoulder.stl" scale="${scale} ${scale} ${scale}"/>
 			</geometry>
 		</collision>
@@ -96,5 +96,5 @@
 			<origin xyz="0 -0.0005 -0.0395" rpy="0 0 0"/>
 			<geometry>
-				<mesh filename="package://hros5_description/meshes/endoskeleton/visual/${side}UpperArm.dae" scale="${scale} ${scale} ${scale}"/>
+				<mesh filename="package://hros5_description/meshes/arms/${side}UpperArm.dae" scale="${scale} ${scale} ${scale}"/>
 			</geometry>
 		</visual>
@@ -102,5 +102,5 @@
 			<origin xyz="0 ${reflect*-0.00025} -0.0395" rpy="0 0 0"/>
 			<geometry>
-				<mesh filename="package://hros5_description/meshes/endoskeleton/collision/${side}UpperArm.stl" scale="${scale} ${scale} ${scale}"/>
+				<mesh filename="package://hros5_description/meshes/arms/${side}UpperArm.stl" scale="${scale} ${scale} ${scale}"/>
 			</geometry>
 		</collision>
@@ -111,5 +111,5 @@
 			<origin xyz="0 ${reflect*-0.003} -0.0204" rpy="0 0 0"/>
 			<geometry>
-				<mesh filename="package://hros5_description/meshes/endoskeleton/visual/${side}LowerArm.dae" scale="${scale} ${scale} ${scale}"/>
+				<mesh filename="package://hros5_description/meshes/arms/${side}LowerArm.dae" scale="${scale} ${scale} ${scale}"/>
 			</geometry>
 		</visual>
@@ -117,5 +117,5 @@
 			<origin xyz="0 ${reflect*-0.003} -0.0204" rpy="0 0 0"/>
 			<geometry>
-				<mesh filename="package://hros5_description/meshes/endoskeleton/collision/${side}LowerArm.stl" scale="${scale} ${scale} ${scale}"/>
+				<mesh filename="package://hros5_description/meshes/arms/${side}LowerArm.stl" scale="${scale} ${scale} ${scale}"/>
 			</geometry>
 		</collision>
@@ -127,5 +127,5 @@
 			<origin xyz="-0.01605 0 -0.008931" rpy="0 0 0"/>
 			<geometry>
-				<mesh filename="package://hros5_description/meshes/endoskeleton/visual/Hip.dae" scale="${scale} ${scale} ${scale}"/>
+				<mesh filename="package://hros5_description/meshes/legs/Hip.dae" scale="${scale} ${scale} ${scale}"/>
 			</geometry>
 		</visual>
@@ -133,5 +133,5 @@
 			<origin xyz="-0.01605 0 -0.008931" rpy="0 0 0"/>
 			<geometry>
-				<mesh filename="package://hros5_description/meshes/endoskeleton/collision/Hip.stl" scale="${scale} ${scale} ${scale}"/>
+				<mesh filename="package://hros5_description/meshes/legs/Hip.stl" scale="${scale} ${scale} ${scale}"/>
 			</geometry>
 		</collision>
@@ -142,5 +142,5 @@
 			<origin xyz="0.077 -0.0052 -0.0041" rpy="0 0 0"/>
 			<geometry>
-				<mesh filename="package://hros5_description/meshes/endoskeleton/visual/HipMotors.dae" scale="${scale} ${scale} ${scale}"/>
+				<mesh filename="package://hros5_description/meshes/legs/HipMotors.dae" scale="${scale} ${scale} ${scale}"/>
 			</geometry>
 		</visual>
@@ -148,5 +148,5 @@
 			<origin xyz="0.077 -0.0052 -0.0041" rpy="0 0 0"/>
 			<geometry>
-				<mesh filename="package://hros5_description/meshes/endoskeleton/collision/HipMotors.stl" scale="${scale} ${scale} ${scale}"/>
+				<mesh filename="package://hros5_description/meshes/legs/HipMotors.stl" scale="${scale} ${scale} ${scale}"/>
 			</geometry>
 		</collision>
@@ -157,5 +157,5 @@
 			<origin xyz="0.001 -0.0095 -0.095" rpy="0 0 0"/>
 			<geometry>
-				<mesh filename="package://hros5_description/meshes/endoskeleton/visual/Thigh.dae" scale="${scale} ${scale} ${scale}"/>
+				<mesh filename="package://hros5_description/meshes/legs/Thigh.dae" scale="${scale} ${scale} ${scale}"/>
 			</geometry>
 		</visual>
@@ -163,5 +163,5 @@
 			<origin xyz="0.001 -0.0095 -0.095" rpy="0 0 0"/>
 			<geometry>
-				<mesh filename="package://hros5_description/meshes/endoskeleton/collision/Thigh.stl" scale="${scale} ${scale} ${scale}"/>
+				<mesh filename="package://hros5_description/meshes/legs/Thigh.stl" scale="${scale} ${scale} ${scale}"/>
 			</geometry>
 		</collision>
@@ -172,5 +172,5 @@
 			<origin xyz="0.004 0 -0.059" rpy="0 0 0"/>
 			<geometry>
-				<mesh filename="package://hros5_description/meshes/endoskeleton/visual/Tibia.dae" scale="${scale} ${scale} ${scale}"/>
+				<mesh filename="package://hros5_description/meshes/legs/Tibia.dae" scale="${scale} ${scale} ${scale}"/>
 			</geometry>
 		</visual>
@@ -178,5 +178,5 @@
 			<origin xyz="0.004 0 -0.059" rpy="0 0 0"/>
 			<geometry>
-				<mesh filename="package://hros5_description/meshes/endoskeleton/collision/Tibia.stl" scale="${scale} ${scale} ${scale}"/>
+				<mesh filename="package://hros5_description/meshes/legs/Tibia.stl" scale="${scale} ${scale} ${scale}"/>
 			</geometry>
 		</collision>
@@ -187,5 +187,5 @@
 			<origin xyz="0.00625 0.00525 0.0042" rpy="0 0 0"/>
 			<geometry>
-				<mesh filename="package://hros5_description/meshes/endoskeleton/visual/Ankle.dae" scale="${scale} ${scale} ${scale}"/>
+				<mesh filename="package://hros5_description/meshes/legs/Ankle.dae" scale="${scale} ${scale} ${scale}"/>
 			</geometry>
 		</visual>
@@ -193,5 +193,5 @@
 			<origin xyz="0.00625 0.00525 0.0042" rpy="0 0 0"/>
 			<geometry>
-				<mesh filename="package://hros5_description/meshes/endoskeleton/collision/Ankle.stl" scale="${scale} ${scale} ${scale}"/>
+				<mesh filename="package://hros5_description/meshes/legs/Ankle.stl" scale="${scale} ${scale} ${scale}"/>
 			</geometry>
 		</collision>
@@ -202,5 +202,5 @@
 			<origin xyz="0.0565 ${reflect*0.007} -0.031" rpy="0 0 0"/>
 			<geometry>
-				<mesh filename="package://hros5_description/meshes/endoskeleton/visual/${side}Foot.dae" scale="${scale} ${scale} ${scale}"/>
+				<mesh filename="package://hros5_description/meshes/legs/${side}Foot.dae" scale="${scale} ${scale} ${scale}"/>
 			</geometry>
 		</visual>
@@ -208,5 +208,5 @@
 			<origin xyz="0.0565 ${reflect*0.007} -0.031" rpy="0 0 0"/>
 			<geometry>
-				<mesh filename="package://hros5_description/meshes/endoskeleton/collision/${side}Foot.stl" scale="${scale} ${scale} ${scale}"/>
+				<mesh filename="package://hros5_description/meshes/legs/${side}Foot.stl" scale="${scale} ${scale} ${scale}"/>
 			</geometry>
 		</collision>

Commit message: Dae for gripper

File: src/hros5_description/urdf/hros5_visuals_collisions_endoskeleton.xacro (robot description, xacro)
@@ -157,5 +157,5 @@
       <origin xyz="0 0 0" rpy="0 0 0"/>
       <geometry>
-        <mesh filename="package://hros5_description/meshes/hands/${side}Gripper.stl" scale="${scale} ${scale} ${scale}"/>
+        <mesh filename="package://hros5_description/meshes/hands/${side}Gripper.dae" scale="${scale} ${scale} ${scale}"/>
       </geometry>
     </visual>

Commit message: dae for hand

File: src/hros5_description/urdf/hros5_visuals_collisions_endoskeleton.xacro (robot description, xacro)
@@ -142,5 +142,5 @@
       <origin xyz="0 0 0" rpy="0 0 0"/>
       <geometry>
-        <mesh filename="package://hros5_description/meshes/hands/${side}Hand.stl" scale="${scale} ${scale} ${scale}"/>
+        <mesh filename="package://hros5_description/meshes/hands/${side}Hand.dae" scale="${scale} ${scale} ${scale}"/>
       </geometry>
     </visual>

Commit message: urdf: add explicit reflect param for foot meshes and add left-hand collision geometry
- foot visuals/collisions macro now takes a reflect parameter; legs forward it so L/R feet mirror y-offset correctly
- added collision meshes to Gazebo left-hand model using existing STL assets (forearm, hand, gripper)

File: src/hros5_description/urdf/hros5_visuals_collisions_endoskeleton.xacro (robot description, xacro)
@@ -244,5 +244,5 @@
 	</xacro:macro>
 	<!-- FOOT VISUALS/COLLISIONS -->
-	<xacro:macro name="visuals_collisions_foot" params="side">
+	<xacro:macro name="visuals_collisions_foot" params="side reflect">
 		<visual>
 			<origin xyz="0.0565 ${reflect*0.007} -0.031" rpy="0 0 0"/>

File: src/hros5_description/urdf/legs/legs.xacro (robot description, xacro)
@@ -85,5 +85,5 @@
 		</joint>
 		<link name="${side}Foot">
-			<xacro:visuals_collisions_foot side="${side}"/>
+			<xacro:visuals_collisions_foot side="${side}" reflect="${reflect}"/>
 			<inertial> <!-- Dummy values from Darwin OP -->
 				<origin xyz="-0.025995 -0.009506 -0.000503" />

File: src/hros5_gazebo/urdf/hands/left_hand_gazebo.xacro (robot description, xacro)
@@ -12,4 +12,9 @@
       </geometry>
     </visual>
+    <collision>
+      <geometry>
+        <mesh filename="package://hros5_description/meshes/hands/LForearm.stl" scale="0.1 0.1 0.1"/>
+      </geometry>
+    </collision>
   </link>
   <!-- Basic link: LHand -->
@@ -20,4 +25,9 @@
       </geometry>
     </visual>
+    <collision>
+      <geometry>
+        <mesh filename="package://hros5_description/meshes/hands/LHand.stl" scale="0.1 0.1 0.1"/>
+      </geometry>
+    </collision>
   </link>
   <!-- Gripper link -->
@@ -28,4 +38,9 @@
       </geometry>
     </visual>
+    <collision>
+      <geometry>
+        <mesh filename="package://hros5_description/meshes/hands/LGripper.stl" scale="0.1 0.1 0.1"/>
+      </geometry>
+    </collision>
   </link>
   <!-- Joint: base_link connects LLowerArm to LHand -->

Commit message: mesh: unify xacro visuals, stl default for gazebo launch and dae for rviz

File: src/hros5_description/urdf/hros5_visuals_collisions_endoskeleton.xacro (robot description, xacro)
@@ -6,5 +6,5 @@
 			<origin xyz="0 0 0" rpy="0 0 0"/>
 			<geometry>
-				<mesh filename="package://hros5_description/meshes/torso/torso.dae" scale="${scale} ${scale} ${scale}"/>
+				<mesh filename="package://hros5_description/meshes/torso/torso.${visual_mesh_ext}" scale="${scale} ${scale} ${scale}"/>
 			</geometry>
 		</visual>
@@ -22,5 +22,5 @@
 			<origin xyz="-0.03 0 0.033" rpy="0 0 0"/>
 			<geometry>
-				<mesh filename="package://hros5_description/meshes/head/LowerHead.dae" scale="${scale} ${scale} ${scale}"/>
+				<mesh filename="package://hros5_description/meshes/head/LowerHead.${visual_mesh_ext}" scale="${scale} ${scale} ${scale}"/>
 			</geometry>
 		</visual>
@@ -37,5 +37,5 @@
 			<origin xyz="0.0075 -0.0045 0.0275" rpy="0 0 0"/>
 			<geometry>
-				<mesh filename="package://hros5_description/meshes/head/UpperHeadBase.dae" scale="${scale} ${scale} ${scale}"/>
+				<mesh filename="package://hros5_description/meshes/head/UpperHeadBase.${visual_mesh_ext}" scale="${scale} ${scale} ${scale}"/>
 			</geometry>
 		</visual>
@@ -51,5 +51,5 @@
 			<origin xyz="-0.03 0 0.00075" rpy="0 0 0"/>
 			<geometry>
-				<mesh filename="package://hros5_description/meshes/head/UpperHeadMotor.dae" scale="${scale} ${scale} ${scale}"/>
+				<mesh filename="package://hros5_description/meshes/head/UpperHeadMotor.${visual_mesh_ext}" scale="${scale} ${scale} ${scale}"/>
 			</geometry>
 		</visual>
@@ -65,5 +65,5 @@
 			<origin xyz="0.001 0 0.0375" rpy="0 0 0"/>
 			<geometry>
-				<mesh filename="package://hros5_description/meshes/head/UpperHeadBack.dae" scale="${scale} ${scale} ${scale}"/>
+				<mesh filename="package://hros5_description/meshes/head/UpperHeadBack.${visual_mesh_ext}" scale="${scale} ${scale} ${scale}"/>
 			</geometry>
 		</visual>
@@ -81,5 +81,5 @@
 			<origin xyz="0 ${reflect*0.0122} -0.0125" rpy="0 0 0"/>
 			<geometry>
-				<mesh filename="package://hros5_description/meshes/arms/${side}Shoulder.dae" scale="${scale} ${scale} ${scale}"/>
+				<mesh filename="package://hros5_description/meshes/arms/${side}Shoulder.${visual_mesh_ext}" scale="${scale} ${scale} ${scale}"/>
 			</geometry>
 		</visual>
@@ -96,5 +96,5 @@
 			<origin xyz="0 -0.0005 -0.0395" rpy="0 0 0"/>
 			<geometry>
-				<mesh filename="package://hros5_description/meshes/arms/${side}UpperArm.dae" scale="${scale} ${scale} ${scale}"/>
+				<mesh filename="package://hros5_description/meshes/arms/${side}UpperArm.${visual_mesh_ext}" scale="${scale} ${scale} ${scale}"/>
 			</geometry>
 		</visual>
@@ -111,5 +111,5 @@
 			<origin xyz="0 ${reflect*-0.003} -0.0204" rpy="0 0 0"/>
 			<geometry>
-				<mesh filename="package://hros5_description/meshes/arms/${side}LowerArm.dae" scale="${scale} ${scale} ${scale}"/>
+				<mesh filename="package://hros5_description/meshes/arms/${side}LowerArm.${visual_mesh_ext}" scale="${scale} ${scale} ${scale}"/>
 			</geometry>
 		</visual>
@@ -127,5 +127,5 @@
       <origin xyz="0 0 0" rpy="0 0 0"/>
       <geometry>
-        <mesh filename="package://hros5_description/meshes/hands/${side}Forearm.dae" scale="${scale} ${scale} ${scale}"/>
+        <mesh filename="package://hros5_description/meshes/hands/${side}Forearm.${visual_mesh_ext}" scale="${scale} ${scale} ${scale}"/>
       </geometry>
     </visual>
@@ -142,5 +142,5 @@
       <origin xyz="0 0 0" rpy="0 0 0"/>
       <geometry>
-        <mesh filename="package://hros5_description/meshes/hands/${side}Hand.dae" scale="${scale} ${scale} ${scale}"/>
+        <mesh filename="package://hros5_description/meshes/hands/${side}Hand.${visual_mesh_ext}" scale="${scale} ${scale} ${scale}"/>
       </geometry>
     </visual>
@@ -157,5 +157,5 @@
       <origin xyz="0 0 0" rpy="0 0 0"/>
       <geometry>
-        <mesh filename="package://hros5_description/meshes/hands/${side}Gripper.dae" scale="${scale} ${scale} ${scale}"/>
+        <mesh filename="package://hros5_description/meshes/hands/${side}Gripper.${visual_mesh_ext}" scale="${scale} ${scale} ${scale}"/>
       </geometry>
     </visual>
@@ -173,5 +173,5 @@
 			<origin xyz="-0.01605 0 -0.008931" rpy="0 0 0"/>
 			<geometry>
-				<mesh filename="package://hros5_description/meshes/legs/Hip.dae" scale="${scale} ${scale} ${scale}"/>
+				<mesh filename="package://hros5_description/meshes/legs/Hip.${visual_mesh_ext}" scale="${scale} ${scale} ${scale}"/>
 			</geometry>
 		</visual>
@@ -188,5 +188,5 @@
 			<origin xyz="0.077 -0.0052 -0.0041" rpy="0 0 0"/>
 			<geometry>
-				<mesh filename="package://hros5_description/meshes/legs/HipMotors.dae" scale="${scale} ${scale} ${scale}"/>
+				<mesh filename="package://hros5_description/meshes/legs/HipMotors.${visual_mesh_ext}" scale="${scale} ${scale} ${scale}"/>
 			</geometry>
 		</visual>
@@ -203,5 +203,5 @@
 			<origin xyz="0.001 -0.0095 -0.095" rpy="0 0 0"/>
 			<geometry>
-				<mesh filename="package://hros5_description/meshes/legs/Thigh.dae" scale="${scale} ${scale} ${scale}"/>
+				<mesh filename="package://hros5_description/meshes/legs/Thigh.${visual_mesh_ext}" scale="${scale} ${scale} ${scale}"/>
 			</geometry>
 		</visual>
@@ -218,5 +218,5 @@
 			<origin xyz="0.004 0 -0.059" rpy="0 0 0"/>
 			<geometry>
-				<mesh filename="package://hros5_description/meshes/legs/Tibia.dae" scale="${scale} ${scale} ${scale}"/>
+				<mesh filename="package://hros5_description/meshes/legs/Tibia.${visual_mesh_ext}" scale="${scale} ${scale} ${scale}"/>
 			</geometry>
 		</visual>
@@ -233,5 +233,5 @@
 			<origin xyz="0.00625 0.00525 0.0042" rpy="0 0 0"/>
 			<geometry>
-				<mesh filename="package://hros5_description/meshes/legs/Ankle.dae" scale="${scale} ${scale} ${scale}"/>
+				<mesh filename="package://hros5_description/meshes/legs/Ankle.${visual_mesh_ext}" scale="${scale} ${scale} ${scale}"/>
 			</geometry>
 		</visual>
@@ -248,5 +248,5 @@
 			<origin xyz="0.0565 ${reflect*0.007} -0.031" rpy="0 0 0"/>
 			<geometry>
-				<mesh filename="package://hros5_description/meshes/legs/${side}Foot.dae" scale="${scale} ${scale} ${scale}"/>
+				<mesh filename="package://hros5_description/meshes/legs/${side}Foot.${visual_mesh_ext}" scale="${scale} ${scale} ${scale}"/>
 			</geometry>
 		</visual>

File: src/hros5_description/urdf/robot/robot.xacro (robot description, xacro)
@@ -4,8 +4,10 @@
 	<!-- Argument with fallback -->
 	<xacro:arg name="meshes_xacro_filename" default="$(find hros5_description)/urdf/hros5_visuals_collisions_endoskeleton.xacro"/>
+	<xacro:arg name="visual_mesh_ext" default="stl"/>
 	<xacro:arg name="scale" default="0.1"/>
 	<!-- XACRO PROPERTIES -->
 	<xacro:property name="PI" value="3.14159265359" />
 	<xacro:property name="PI_2" value="1.57079632679" />
+	<xacro:property name="visual_mesh_ext" value="$(arg visual_mesh_ext)" />
 	<xacro:property name="scale" value="$(arg scale)" />
  <!-- Include shared geometry macros -->
