Commit message: Only launch arms, not torso

File: src/hros5_description/urdf/arms/arms_test.xacro (robot description, xacro)
@@ -10,5 +10,13 @@
 	<xacro:include filename="$(arg meshes_xacro_filename)" />
 	<!-- Load xacro subparts of the robot -->
-	<xacro:include filename="$(find hros5_description)/urdf/torso/torso.xacro" />
+	<!--xacro:include filename="$(find hros5_description)/urdf/torso/torso.xacro" /-->
   <xacro:include filename="$(find hros5_description)/urdf/arms/arms.xacro"/>
+	<!-- Anchor link -->
+  <link name="base_link"/>
+  <link name="torso"/>
+  <joint name="base_to_torso" type="fixed">
+    <parent link="base_link"/>
+    <child link="torso"/>
+    <origin xyz="0 0 0" rpy="0 0 0"/>
+  </joint>
 </robot>

Commit message: Left hand is now part of robot!

File: src/hros5_description/urdf/arms/arms_test.xacro (robot description, xacro)
@@ -12,4 +12,5 @@
 	<!--xacro:include filename="$(find hros5_description)/urdf/torso/torso.xacro" /-->
   <xacro:include filename="$(find hros5_description)/urdf/arms/arms.xacro"/>
+	<xacro:include filename="$(find hros5_description)/urdf/hands/hands.xacro" />
 	<!-- Anchor link -->
   <link name="base_link"/>

File: src/hros5_description/urdf/hands/hands.xacro (robot description, xacro)
@@ -5,5 +5,5 @@
       <parent link="${side}LowerArm"/>
       <child link="${side}Forearm"/>
-      <origin xyz="0 0 0" rpy="0 0 0"/>
+      <origin xyz="0 0 -0.075" rpy="-1.5708 3.1416 0"/>
     </joint>
     <link name="${side}Forearm">
@@ -38,5 +38,5 @@
     <parent link="LForearm"/>
     <child link="LHand"/>
-    <origin xyz="0 0 0.05" rpy="0 0 0"/>
+    <origin xyz="0 -0.0205 0" rpy="-3.0949 0 -1.5708" />
     <axis xyz="1 0 0"/>
     <limit lower="-3.14" upper="3.14" effort="1.0" velocity="1.0"/>
@@ -45,21 +45,21 @@
     <parent link="RForearm"/>
     <child link="RHand"/>
-    <origin xyz="0 0 0.05" rpy="0 0 0"/>
+    <origin xyz="0 -0.0205 0" rpy="-3.0949 0 -1.5708" />
     <axis xyz="1 0 0"/>
-    <limit lower="-1.57" upper="1.57" effort="1.0" velocity="1.0"/>
+    <limit lower="-3.14" upper="3.14" effort="1.0" velocity="1.0"/>
   </joint-->
   <joint name="LGripper" type="revolute">
     <parent link="LHand"/>
     <child link="LGripper"/>
-    <origin xyz="0 0 0.05" rpy="0 0 0"/>
-    <axis xyz="0 1 0"/>
-    <limit lower="0.0" upper="0.8" effort="1.0" velocity="1.0"/>
+    <origin xyz="0.021 0.008 -0.0205" rpy="-1.5708 -1.5708 1.5708" />
+    <axis xyz="1 0 0"/>
+    <limit lower="-1.0" upper="0.5" effort="1.0" velocity="1.0"/>
   </joint>
   <!--joint name="RGripper" type="revolute">
     <parent link="RHand"/>
     <child link="RGripper"/>
-    <origin xyz="0 0 0.05" rpy="0 0 0"/>
-    <axis xyz="0 1 0"/>
-    <limit lower="0.0" upper="0.8" effort="1.0" velocity="1.0"/>
+    <origin xyz="0.021 0.008 -0.0205" rpy="-1.5708 -1.5708 1.5708" />
+    <axis xyz="1 0 0"/>
+    <limit lower="-1.0" upper="0.5" effort="1.0" velocity="1.0"/>
   </joint-->
 </robot>

File: src/hros5_description/urdf/hands/hands_test.xacro (robot description, xacro)
@@ -18,5 +18,5 @@
     <parent link="base_link"/>
     <child link="LLowerArm"/>
-    <origin xyz="0 0 0" rpy="0 0 0"/>
+    <origin xyz="0 0 0.075" rpy="0.0 -1.5708 0"/>
   </joint>
   <!--link name="RLowerArm"/>
@@ -24,5 +24,5 @@
     <parent link="base_link"/>
     <child link="RLowerArm"/>
-    <origin xyz="0 0 0" rpy="0 0 0"/>
+    <origin xyz="0 0 0.075" rpy="0.0 -1.5708 0"/>
   </joint-->
 </robot>

File: src/hros5_description/urdf/hros5_visuals_collisions_endoskeleton.xacro (robot description, xacro)
@@ -125,5 +125,5 @@
   <xacro:macro name="visuals_collisions_forearm" params="side reflect">
     <visual>
-      <origin xyz="0 ${reflect*-0.003} -0.0204" rpy="1.5708 -1.5708 0"/>
+      <origin xyz="0 0 0" rpy="0 0 0"/>
       <geometry>
         <mesh filename="package://hros5_description/meshes/hands/${side}Forearm.stl" scale="${scale} ${scale} ${scale}"/>
@@ -131,5 +131,5 @@
     </visual>
     <collision>
-      <origin xyz="0 ${reflect*-0.003} -0.0204" rpy="1.5708 -1.5708 0"/>
+      <origin xyz="0 0 0" rpy="0 0 0"/>
       <geometry>
         <mesh filename="package://hros5_description/meshes/hands/${side}Forearm.stl" scale="${scale} ${scale} ${scale}"/>
@@ -140,5 +140,5 @@
   <xacro:macro name="visuals_collisions_hand" params="side reflect">
     <visual>
-      <origin xyz="0 0 0.05" rpy="1.5708 0 0"/>
+      <origin xyz="0 0 0" rpy="0 0 0"/>
       <geometry>
         <mesh filename="package://hros5_description/meshes/hands/${side}Hand.stl" scale="${scale} ${scale} ${scale}"/>
@@ -146,5 +146,5 @@
     </visual>
     <collision>
-      <origin xyz="0 0 0.05" rpy="1.5708 0 0"/>
+      <origin xyz="0 0 0" rpy="0 0 0"/>
       <geometry>
         <mesh filename="package://hros5_description/meshes/hands/${side}Hand.stl" scale="${scale} ${scale} ${scale}"/>
@@ -155,5 +155,5 @@
   <xacro:macro name="visuals_collisions_gripper" params="side reflect">
     <visual>
-      <origin xyz="0 0 0.05" rpy="1.5708 0 -1.5708"/>
+      <origin xyz="0 0 0" rpy="0 0 0"/>
       <geometry>
         <mesh filename="package://hros5_description/meshes/hands/${side}Gripper.stl" scale="${scale} ${scale} ${scale}"/>
@@ -161,5 +161,5 @@
     </visual>
     <collision>
-      <origin xyz="0 0 0.05" rpy="1.5708 0 -1.5708"/>
+      <origin xyz="0 0 0" rpy="0 0 0"/>
       <geometry>
         <mesh filename="package://hros5_description/meshes/hands/${side}Gripper.stl" scale="${scale} ${scale} ${scale}"/>

File: src/hros5_description/urdf/robot/robot.xacro (robot description, xacro)
@@ -14,5 +14,5 @@
 	<xacro:include filename="$(find hros5_description)/urdf/head/head.xacro" />
 	<xacro:include filename="$(find hros5_description)/urdf/arms/arms.xacro" />
-	<!-- <xacro:include filename="$(find hros5_description)/urdf/hands/hands.xacro" /> -->
+	<xacro:include filename="$(find hros5_description)/urdf/hands/hands.xacro" />
 	<xacro:include filename="$(find hros5_description)/urdf/legs/legs.xacro" />
 	<!-- <xacro:include filename="$(find hros5_description)/urdf/modules/imu.xacro" />
