Commit message: Added model file for mx28at
move to /dynamixel hw interface param dxl model

File: src/hros5_demos/urdf/test_urdf.xacro (robot description, xacro)
@@ -18,4 +18,20 @@
     <limit lower="-1.57" upper="1.57" effort="1.0" velocity="1.0"/>
   </joint>
+<ros2_control name="DynamixelHardware" type="system">
+  <hardware>
+    <plugin>dynamixel_hardware_interface/DynamixelHardware</plugin>
+    <param name="serial_port">/dev/ttyUSB0</param>
+    <param name="baud_rate">1000000</param>
+    <param name="protocol_version">2.0</param>
+    <param name="joint_ids">22,24</param>
+    <param name="joint_names">LHand,LGripper</param>
+    <param name="error_timeout_ms">100</param>
+    <param name="number_of_transmissions">2</param>
+    <param name="dynamixel_state_pub_msg_name">dynamixel_hardware_interface/dxl_state</param>
+    <param name="get_dynamixel_data_srv_name">dynamixel_hardware_interface/get_dxl_data</param>
+    <param name="set_dynamixel_data_srv_name">dynamixel_hardware_interface/set_dxl_data</param>
+    <param name="reboot_dxl_srv_name">dynamixel_hardware_interface/reboot_dxl</param>
+    <param name="set_dxl_torque_srv_name">dynamixel_hardware_interface/set_dxl_torque</param>
+  </hardware>
   <gpio name="dxl1">
     <param name="type">dxl</param>
@@ -25,8 +41,8 @@
     <state_interface name="Present Velocity"/>
     <state_interface name="Present Current"/>
-    <param name="Position P Gain">800</param> <!-- Proportional gain for position control -->
-    <param name="Position I Gain">100</param> <!-- Integral gain for position control -->
-    <param name="Position D Gain">100</param> <!-- Derivative gain for position control -->
-    <param name="Drive Mode">0</param> <!-- 0: Clockwise, 1: Counterclockwise -->
+    <param name="Position P Gain">800</param>
+    <param name="Position I Gain">100</param>
+    <param name="Position D Gain">100</param>
+    <param name="Drive Mode">0</param>
   </gpio>
   <gpio name="dxl2">
@@ -37,8 +53,21 @@
     <state_interface name="Present Velocity"/>
     <state_interface name="Present Current"/>
-    <param name="Position P Gain">800</param> <!-- Proportional gain for position control -->
-    <param name="Position I Gain">100</param> <!-- Integral gain for position control -->
-    <param name="Position D Gain">100</param> <!-- Derivative gain for position control -->
-    <param name="Drive Mode">0</param> <!-- 0: Clockwise, 1: Counterclockwise -->
+    <param name="Position P Gain">800</param>
+    <param name="Position I Gain">100</param>
+    <param name="Position D Gain">100</param>
+    <param name="Drive Mode">0</param>
   </gpio>
+  <joint name="LHand">
+    <command_interface name="position"/>
+    <state_interface name="position"/>
+    <state_interface name="velocity"/>
+    <state_interface name="effort"/>
+  </joint>
+  <joint name="LGripper">
+    <command_interface name="position"/>
+    <state_interface name="position"/>
+    <state_interface name="velocity"/>
+    <state_interface name="effort"/>
+  </joint>
+</ros2_control>
 </robot>
