Commit message: Display hands in rviz
Trying to get the hands to show up in rviz, made a launch file for arms(and torso) that finally works. Need to get the hands up as well

File: src/hros5_description/urdf/hands/hands.xacro (robot description, xacro)
@@ -1,25 +1,49 @@
 <?xml version="1.0"?>
-<robot xmlns:xacro="http://ros.org/wiki/xacro">
-  <xacro:macro name="hands" params="">
-    <!-- Links -->
-    <link name="l_hand_link"/>
-    <link name="l_gripper_link"/>
-    <!-- Joints -->
-    <!-- LHand joint -->
-    <joint name="LHand" type="revolute">
-      <parent link="l_forearm_link"/>
-      <child link="l_hand_link"/>
-      <origin xyz="0 0 0.02" rpy="0 0 0"/>
+<robot xmlns:xacro="http://www.ros.org/wiki/xacro">
+  <xacro:macro name="hands_links_joints" params="side reflect">
+    <joint name="${side}ForearmJoint" type="fixed">
+      <parent link="${side}LowerArm"/>
+      <child link="${side}Forearm"/>
+      <origin xyz="0 0 0" rpy="0 0 0"/>
+    </joint>
+    <link name="${side}Forearm">
+      <xacro:visuals_collisions_hand_section side="${side}" reflect="${reflect}"/>
+      <inertial>
+        <origin xyz="0 0 0"/>
+        <mass value="0.1"/>
+        <inertia ixx="0.001" ixy="0.0" ixz="0.0" iyy="0.001" iyz="0.0" izz="0.001"/>
+      </inertial>
+    </link>
+    <joint name="${side}Wrist" type="revolute">
+      <parent link="${side}Forearm"/>
+      <child link="${side}Hand"/>
+      <origin xyz="0 0 0.05" rpy="0 0 0"/>
       <axis xyz="0 0 1"/>
-      <limit lower="-3.14" upper="3.14" effort="1.0" velocity="1.0"/>
+      <limit lower="-1.57" upper="1.57" effort="1.0" velocity="1.0"/>
     </joint>
-    <!-- LGripper joint -->
-    <joint name="LGripper" type="revolute">
-      <parent link="l_hand_link"/>
-      <child link="l_gripper_link"/>
-      <origin xyz="0 0 0.02" rpy="0 0 0"/>
-      <axis xyz="0 1 0"/>
-      <limit lower="0.0" upper="1.0" effort="1.0" velocity="1.0"/>
+    <link name="${side}Hand">
+      <inertial>
+        <origin xyz="0 0 0"/>
+        <mass value="0.08"/>
+        <inertia ixx="0.0008" ixy="0.0" ixz="0.0" iyy="0.0008" iyz="0.0" izz="0.0008"/>
+      </inertial>
+    </link>
+    <joint name="${side}Gripper" type="revolute">
+      <parent link="${side}Hand"/>
+      <child link="${side}Gripper"/>
+      <origin xyz="0 0 0.05" rpy="0 0 0"/>
+      <axis xyz="0 0 1"/>
+      <limit lower="0.0" upper="0.8" effort="1.0" velocity="1.0"/>
     </joint>
+    <link name="${side}Gripper">
+      <inertial>
+        <origin xyz="0 0 0"/>
+        <mass value="0.05"/>
+        <inertia ixx="0.0005" ixy="0.0" ixz="0.0" iyy="0.0005" iyz="0.0" izz="0.0005"/>
+      </inertial>
+    </link>
   </xacro:macro>
+  <!-- Direct test instantiation -->
+  <xacro:hands_links_joints side="L" reflect="1"/>
+  <!--xacro:hands_links_joints side="R" reflect="-1"/-->
 </robot>

File: src/hros5_description/urdf/hros5_visuals_collisions_endoskeleton.xacro (robot description, xacro)
@@ -121,4 +121,46 @@
 		</collision>
 	</xacro:macro>
+	 <!-- Meshes for the forearm, wrist, hand, and gripper -->
+  <xacro:macro name="visuals_collisions_hand_section" params="side reflect">
+    <!-- Forearm mesh (lower part, if different from existing lower arm) -->
+    <visual>
+      <origin xyz="0 ${reflect*-0.003} -0.0204" rpy="0 0 0"/>
+      <geometry>
+        <mesh filename="package://hros5_description/meshes/hands/${side}Forearm.stl" scale="${scale} ${scale} ${scale}"/>
+      </geometry>
+    </visual>
+    <collision>
+      <origin xyz="0 ${reflect*-0.003} -0.0204" rpy="0 0 0"/>
+      <geometry>
+        <mesh filename="package://hros5_description/meshes/hands/${side}Forearm.stl" scale="${scale} ${scale} ${scale}"/>
+      </geometry>
+    </collision>
+    <!-- Hand -->
+    <visual>
+      <origin xyz="0 0 0.05" rpy="0 0 0"/>
+      <geometry>
+        <mesh filename="package://hros5_description/meshes/hands/${side}Hand.stl" scale="${scale} ${scale} ${scale}"/>
+      </geometry>
+    </visual>
+    <collision>
+      <origin xyz="0 0 0.05" rpy="0 0 0"/>
+      <geometry>
+        <mesh filename="package://hros5_description/meshes/hands/${side}Hand.stl" scale="${scale} ${scale} ${scale}"/>
+      </geometry>
+    </collision>
+    <!-- Gripper -->
+    <visual>
+      <origin xyz="0 0 0.05" rpy="0 0 0"/>
+      <geometry>
+        <mesh filename="package://hros5_description/meshes/hands/${side}Gripper.stl" scale="${scale} ${scale} ${scale}"/>
+      </geometry>
+    </visual>
+    <collision>
+      <origin xyz="0 0 0.05" rpy="0 0 0"/>
+      <geometry>
+        <mesh filename="package://hros5_description/meshes/hands/${side}Gripper.stl" scale="${scale} ${scale} ${scale}"/>
+      </geometry>
+    </collision>
+  </xacro:macro>
 <!-- LEGS VISUALS/COLLISIONS -->
 	<!-- HIP VISUALS/COLLISIONS -->

Commit message: Hand shows up and moves in rviz

File: src/hros5_description/urdf/hands/hands.xacro (robot description, xacro)
@@ -8,42 +8,58 @@
     </joint>
     <link name="${side}Forearm">
-      <xacro:visuals_collisions_hand_section side="${side}" reflect="${reflect}"/>
+      <xacro:visuals_collisions_forearm side="${side}" reflect="${reflect}"/>
       <inertial>
-        <origin xyz="0 0 0"/>
+        <origin xyz="0 0 0" />
         <mass value="0.1"/>
         <inertia ixx="0.001" ixy="0.0" ixz="0.0" iyy="0.001" iyz="0.0" izz="0.001"/>
       </inertial>
     </link>
-    <joint name="${side}Wrist" type="revolute">
-      <parent link="${side}Forearm"/>
-      <child link="${side}Hand"/>
-      <origin xyz="0 0 0.05" rpy="0 0 0"/>
-      <axis xyz="0 0 1"/>
-      <limit lower="-1.57" upper="1.57" effort="1.0" velocity="1.0"/>
-    </joint>
     <link name="${side}Hand">
-      <inertial>
-        <origin xyz="0 0 0"/>
-        <mass value="0.08"/>
-        <inertia ixx="0.0008" ixy="0.0" ixz="0.0" iyy="0.0008" iyz="0.0" izz="0.0008"/>
-      </inertial>
+      <xacro:visuals_collisions_hand side="${side}" reflect="${reflect}"/>
+        <inertial>
+          <origin xyz="0 0 0"/>
+          <mass value="0.08"/>
+          <inertia ixx="0.0008" ixy="0.0" ixz="0.0" iyy="0.0008" iyz="0.0" izz="0.0008"/>
+        </inertial>
     </link>
-    <joint name="${side}Gripper" type="revolute">
-      <parent link="${side}Hand"/>
-      <child link="${side}Gripper"/>
-      <origin xyz="0 0 0.05" rpy="0 0 0"/>
-      <axis xyz="0 0 1"/>
-      <limit lower="0.0" upper="0.8" effort="1.0" velocity="1.0"/>
-    </joint>
     <link name="${side}Gripper">
-      <inertial>
-        <origin xyz="0 0 0"/>
-        <mass value="0.05"/>
-        <inertia ixx="0.0005" ixy="0.0" ixz="0.0" iyy="0.0005" iyz="0.0" izz="0.0005"/>
-      </inertial>
+      <xacro:visuals_collisions_gripper side="${side}" reflect="${reflect}"/>
+        <inertial>
+          <origin xyz="0 0 0"/>
+          <mass value="0.05"/>
+          <inertia ixx="0.0005" ixy="0.0" ixz="0.0" iyy="0.0005" iyz="0.0" izz="0.0005"/>
+        </inertial>
     </link>
   </xacro:macro>
   <!-- Direct test instantiation -->
-  <xacro:hands_links_joints side="L" reflect="1"/>
-  <!--xacro:hands_links_joints side="R" reflect="-1"/-->
+  <xacro:hands_links_joints reflect="1" side="L"/>
+  <!--xacro:hands_links_joints reflect="-1" side="R"/-->
+  <joint name="LWrist" type="revolute">
+    <parent link="LForearm"/>
+    <child link="LHand"/>
+    <origin xyz="0 0 0.05" rpy="0 0 0"/>
+    <axis xyz="1 0 0"/>
+    <limit lower="-3.14" upper="3.14" effort="1.0" velocity="1.0"/>
+  </joint>
+  <!--joint name="RWrist" type="revolute">
+    <parent link="RForearm"/>
+    <child link="RHand"/>
+    <origin xyz="0 0 0.05" rpy="0 0 0"/>
+    <axis xyz="1 0 0"/>
+    <limit lower="-1.57" upper="1.57" effort="1.0" velocity="1.0"/>
+  </joint-->
+  <joint name="LGripper" type="revolute">
+    <parent link="LHand"/>
+    <child link="LGripper"/>
+    <origin xyz="0 0 0.05" rpy="0 0 0"/>
+    <axis xyz="0 1 0"/>
+    <limit lower="0.0" upper="0.8" effort="1.0" velocity="1.0"/>
+  </joint>
+  <!--joint name="RGripper" type="revolute">
+    <parent link="RHand"/>
+    <child link="RGripper"/>
+    <origin xyz="0 0 0.05" rpy="0 0 0"/>
+    <axis xyz="0 1 0"/>
+    <limit lower="0.0" upper="0.8" effort="1.0" velocity="1.0"/>
+  </joint-->
 </robot>

File: src/hros5_description/urdf/hros5_visuals_collisions_endoskeleton.xacro (robot description, xacro)
@@ -121,9 +121,9 @@
 		</collision>
 	</xacro:macro>
-	 <!-- Meshes for the forearm, wrist, hand, and gripper -->
-  <xacro:macro name="visuals_collisions_hand_section" params="side reflect">
-    <!-- Forearm mesh (lower part, if different from existing lower arm) -->
+<!-- HANDS VISUALS/COLLISIONS -->
+  <!-- FOREARM VISUALS/COLLISIONS -->
+  <xacro:macro name="visuals_collisions_forearm" params="side reflect">
     <visual>
-      <origin xyz="0 ${reflect*-0.003} -0.0204" rpy="0 0 0"/>
+      <origin xyz="0 ${reflect*-0.003} -0.0204" rpy="1.5708 -1.5708 0"/>
       <geometry>
         <mesh filename="package://hros5_description/meshes/hands/${side}Forearm.stl" scale="${scale} ${scale} ${scale}"/>
@@ -131,12 +131,14 @@
     </visual>
     <collision>
-      <origin xyz="0 ${reflect*-0.003} -0.0204" rpy="0 0 0"/>
+      <origin xyz="0 ${reflect*-0.003} -0.0204" rpy="1.5708 -1.5708 0"/>
       <geometry>
         <mesh filename="package://hros5_description/meshes/hands/${side}Forearm.stl" scale="${scale} ${scale} ${scale}"/>
       </geometry>
     </collision>
-    <!-- Hand -->
+  </xacro:macro>
+  <!-- HAND VISUALS/COLLISIONS -->
+  <xacro:macro name="visuals_collisions_hand" params="side reflect">
     <visual>
-      <origin xyz="0 0 0.05" rpy="0 0 0"/>
+      <origin xyz="0 0 0.05" rpy="1.5708 0 0"/>
       <geometry>
         <mesh filename="package://hros5_description/meshes/hands/${side}Hand.stl" scale="${scale} ${scale} ${scale}"/>
@@ -144,12 +146,14 @@
     </visual>
     <collision>
-      <origin xyz="0 0 0.05" rpy="0 0 0"/>
+      <origin xyz="0 0 0.05" rpy="1.5708 0 0"/>
       <geometry>
         <mesh filename="package://hros5_description/meshes/hands/${side}Hand.stl" scale="${scale} ${scale} ${scale}"/>
       </geometry>
     </collision>
-    <!-- Gripper -->
+  </xacro:macro>
+  <!-- GRIPPER VISUALS/COLLISIONS -->
+  <xacro:macro name="visuals_collisions_gripper" params="side reflect">
     <visual>
-      <origin xyz="0 0 0.05" rpy="0 0 0"/>
+      <origin xyz="0 0 0.05" rpy="1.5708 0 -1.5708"/>
       <geometry>
         <mesh filename="package://hros5_description/meshes/hands/${side}Gripper.stl" scale="${scale} ${scale} ${scale}"/>
@@ -157,5 +161,5 @@
     </visual>
     <collision>
-      <origin xyz="0 0 0.05" rpy="0 0 0"/>
+      <origin xyz="0 0 0.05" rpy="1.5708 0 -1.5708"/>
       <geometry>
         <mesh filename="package://hros5_description/meshes/hands/${side}Gripper.stl" scale="${scale} ${scale} ${scale}"/>

Commit message: Both hands part of robot!

File: src/hros5_description/urdf/hands/hands.xacro (robot description, xacro)
@@ -34,5 +34,5 @@
   <!-- Direct test instantiation -->
   <xacro:hands_links_joints reflect="1" side="L"/>
-  <!--xacro:hands_links_joints reflect="-1" side="R"/-->
+  <xacro:hands_links_joints reflect="-1" side="R"/>
   <joint name="LWrist" type="revolute">
     <parent link="LForearm"/>
@@ -42,5 +42,5 @@
     <limit lower="-3.14" upper="3.14" effort="1.0" velocity="1.0"/>
   </joint>
-  <!--joint name="RWrist" type="revolute">
+  <joint name="RWrist" type="revolute">
     <parent link="RForearm"/>
     <child link="RHand"/>
@@ -48,5 +48,5 @@
     <axis xyz="1 0 0"/>
     <limit lower="-3.14" upper="3.14" effort="1.0" velocity="1.0"/>
-  </joint-->
+  </joint>
   <joint name="LGripper" type="revolute">
     <parent link="LHand"/>
@@ -56,5 +56,5 @@
     <limit lower="-1.0" upper="0.5" effort="1.0" velocity="1.0"/>
   </joint>
-  <!--joint name="RGripper" type="revolute">
+  <joint name="RGripper" type="revolute">
     <parent link="RHand"/>
     <child link="RGripper"/>
@@ -62,4 +62,4 @@
     <axis xyz="1 0 0"/>
     <limit lower="-1.0" upper="0.5" effort="1.0" velocity="1.0"/>
-  </joint-->
+  </joint>
 </robot>

File: src/hros5_description/urdf/hands/hands_test.xacro (robot description, xacro)
@@ -18,11 +18,11 @@
     <parent link="base_link"/>
     <child link="LLowerArm"/>
-    <origin xyz="0 0 0.075" rpy="0.0 -1.5708 0"/>
+    <origin xyz="0 0.1 0.075" rpy="0.0 -1.5708 0"/>
   </joint>
-  <!--link name="RLowerArm"/>
+  <link name="RLowerArm"/>
   <joint name="base_to_rlowerarm" type="fixed">
     <parent link="base_link"/>
     <child link="RLowerArm"/>
-    <origin xyz="0 0 0.075" rpy="0.0 -1.5708 0"/>
-  </joint-->
+    <origin xyz="0 -0.1 0.075" rpy="0.0 -1.5708 0"/>
+  </joint>
 </robot>

File: src/hros5_description/urdf/hros5_visuals_collisions_endoskeleton.xacro (robot description, xacro)
@@ -127,5 +127,5 @@
       <origin xyz="0 0 0" rpy="0 0 0"/>
       <geometry>
-        <mesh filename="package://hros5_description/meshes/hands/${side}Forearm.stl" scale="${scale} ${scale} ${scale}"/>
+        <mesh filename="package://hros5_description/meshes/hands/${side}Forearm.dae" scale="${scale} ${scale} ${scale}"/>
       </geometry>
     </visual>

Commit message: Messed up some joint/link names
The joints are wrist and grip, while the links are hand and gripper

File: src/hros5_description/urdf/hands/hands.xacro (robot description, xacro)
@@ -49,5 +49,5 @@
     <limit lower="-3.14" upper="3.14" effort="1.0" velocity="1.0"/>
   </joint>
-  <joint name="LGripper" type="revolute">
+  <joint name="LGrip" type="revolute">
     <parent link="LHand"/>
     <child link="LGripper"/>
@@ -56,5 +56,5 @@
     <limit lower="-1.0" upper="0.5" effort="1.0" velocity="1.0"/>
   </joint>
-  <joint name="RGripper" type="revolute">
+  <joint name="RGrip" type="revolute">
     <parent link="RHand"/>
     <child link="RGripper"/>

File: src/hros5_description/urdf/hands/left_hand.xacro (robot description, xacro)
@@ -41,5 +41,5 @@
     <limit lower="-3.14" upper="3.14" effort="1.0" velocity="1.0"/>
   </joint>
-  <joint name="LGripper" type="revolute">
+  <joint name="LGrip" type="revolute">
     <parent link="LHand"/>
     <child link="LGripper"/>
