Commit message: urdf: strip ros2_control and transmission tags from component xacros and centralize config in hros5_control.xacro
- removed all <transmission> and ros2_control / gazebo-plugin tags from component xacros (head, arms, legs, hands, torso)
- moved remaining hardwareInterface definitions into hros5_control.xacro
- kept component xacros focused on kinematics + visuals/collisions only

Fixes #10

File: src/hros5_description/urdf/hands/hands_control.xacro (robot description, xacro)
@@ -1,20 +1,4 @@
 <?xml version="1.0"?>
 <robot xmlns:xacro="http://www.ros.org/wiki/xacro">
-  <xacro:macro name="hands_control" params="">
-    <ros2_control name="DynamixelHardware" type="system">
-      <hardware>
-        <plugin>dynamixel_hardware_interface/DynamixelHardware</plugin>
-      </hardware>
-      <joint name="LHand">
-        <command_interface name="position"/>
-        <state_interface name="position"/>
-        <state_interface name="velocity"/>
-      </joint>
-      <joint name="LGripper">
-        <command_interface name="position"/>
-        <state_interface name="position"/>
-        <state_interface name="velocity"/>
-      </joint>
-    </ros2_control>
-  </xacro:macro>
+  <!-- ros2_control for the hands now lives in urdf/hros5_control.xacro -->
 </robot>

File: src/hros5_description/urdf/hros5.urdf (robot description, URDF)
Before this commit: robot hros5, 31 links, 30 joints
Links:
- added link LForearm, mass 0.1; collision mesh filename=package://hros5_description/meshes/hands/LForearm.stl scale=0.1 0.1 0.1; visual mesh filename=package://hros5_description/meshes/hands/LForearm.dae scale=0.1 0.1 0.1
- added link LGripper, mass 0.05; collision mesh filename=package://hros5_description/meshes/hands/LGripper.stl scale=0.1 0.1 0.1; visual mesh filename=package://hros5_description/meshes/hands/LGripper.dae scale=0.1 0.1 0.1
- added link LHand, mass 0.08; collision mesh filename=package://hros5_description/meshes/hands/LHand.stl scale=0.1 0.1 0.1; visual mesh filename=package://hros5_description/meshes/hands/LHand.dae scale=0.1 0.1 0.1
- added link RForearm, mass 0.1; collision mesh filename=package://hros5_description/meshes/hands/RForearm.stl scale=0.1 0.1 0.1; visual mesh filename=package://hros5_description/meshes/hands/RForearm.dae scale=0.1 0.1 0.1
- added link RGripper, mass 0.05; collision mesh filename=package://hros5_description/meshes/hands/RGripper.stl scale=0.1 0.1 0.1; visual mesh filename=package://hros5_description/meshes/hands/RGripper.dae scale=0.1 0.1 0.1
- added link RHand, mass 0.08; collision mesh filename=package://hros5_description/meshes/hands/RHand.stl scale=0.1 0.1 0.1; visual mesh filename=package://hros5_description/meshes/hands/RHand.dae scale=0.1 0.1 0.1
- link LAnkle: geometry collision mesh filename=package://hros5_description/meshes/legs/Ankle.stl scale=0.1 0.1 0.1; visual mesh filename=package://hros5_description/meshes/legs/Ankle.dae scale=0.1 0.1 0.1
- link LFoot: geometry collision mesh filename=package://hros5_description/meshes/legs/LFoot.stl scale=0.1 0.1 0.1; visual mesh filename=package://hros5_description/meshes/legs/LFoot.dae scale=0.1 0.1 0.1
- link LHip: geometry collision mesh filename=package://hros5_description/meshes/legs/Hip.stl scale=0.1 0.1 0.1; visual mesh filename=package://hros5_description/meshes/legs/Hip.dae scale=0.1 0.1 0.1
- link LHipMotors: geometry collision mesh filename=package://hros5_description/meshes/legs/HipMotors.stl scale=0.1 0.1 0.1; visual mesh filename=package://hros5_description/meshes/legs/HipMotors.dae scale=0.1 0.1 0.1
- link LLowerArm: geometry collision mesh filename=package://hros5_description/meshes/arms/LLowerArm.stl scale=0.1 0.1 0.1; visual mesh filename=package://hros5_description/meshes/arms/LLowerArm.dae scale=0.1 0.1 0.1
- link LShoulder: geometry collision mesh filename=package://hros5_description/meshes/arms/LShoulder.stl scale=0.1 0.1 0.1; visual mesh filename=package://hros5_description/meshes/arms/LShoulder.dae scale=0.1 0.1 0.1
- link LThigh: geometry collision mesh filename=package://hros5_description/meshes/legs/Thigh.stl scale=0.1 0.1 0.1; visual mesh filename=package://hros5_description/meshes/legs/Thigh.dae scale=0.1 0.1 0.1
- link LTibia: geometry collision mesh filename=package://hros5_description/meshes/legs/Tibia.stl scale=0.1 0.1 0.1; visual mesh filename=package://hros5_description/meshes/legs/Tibia.dae scale=0.1 0.1 0.1
- link LUpperArm: geometry collision mesh filename=package://hros5_description/meshes/arms/LUpperArm.stl scale=0.1 0.1 0.1; visual mesh filename=package://hros5_description/meshes/arms/LUpperArm.dae scale=0.1 0.1 0.1
- link LowerHead: geometry collision mesh filename=package://hros5_description/meshes/head/LowerHead.stl scale=0.1 0.1 0.1; visual mesh filename=package://hros5_description/meshes/head/LowerHead.dae scale=0.1 0.1 0.1
- link RAnkle: geometry collision mesh filename=package://hros5_description/meshes/legs/Ankle.stl scale=0.1 0.1 0.1; visual mesh filename=package://hros5_description/meshes/legs/Ankle.dae scale=0.1 0.1 0.1
- link RFoot: geometry collision mesh filename=package://hros5_description/meshes/legs/RFoot.stl scale=0.1 0.1 0.1; visual mesh filename=package://hros5_description/meshes/legs/RFoot.dae scale=0.1 0.1 0.1
- link RHip: geometry collision mesh filename=package://hros5_description/meshes/legs/Hip.stl scale=0.1 0.1 0.1; visual mesh filename=package://hros5_description/meshes/legs/Hip.dae scale=0.1 0.1 0.1
- link RHipMotors: geometry collision mesh filename=package://hros5_description/meshes/legs/HipMotors.stl scale=0.1 0.1 0.1; visual mesh filename=package://hros5_description/meshes/legs/HipMotors.dae scale=0.1 0.1 0.1
- link RLowerArm: geometry collision mesh filename=package://hros5_description/meshes/arms/RLowerArm.stl scale=0.1 0.1 0.1; visual mesh filename=package://hros5_description/meshes/arms/RLowerArm.dae scale=0.1 0.1 0.1
- link RShoulder: geometry collision mesh filename=package://hros5_description/meshes/arms/RShoulder.stl scale=0.1 0.1 0.1; visual mesh filename=package://hros5_description/meshes/arms/RShoulder.dae scale=0.1 0.1 0.1
- link RThigh: geometry collision mesh filename=package://hros5_description/meshes/legs/Thigh.stl scale=0.1 0.1 0.1; visual mesh filename=package://hros5_description/meshes/legs/Thigh.dae scale=0.1 0.1 0.1
- link RTibia: geometry collision mesh filename=package://hros5_description/meshes/legs/Tibia.stl scale=0.1 0.1 0.1; visual mesh filename=package://hros5_description/meshes/legs/Tibia.dae scale=0.1 0.1 0.1
- link RUpperArm: geometry collision mesh filename=package://hros5_description/meshes/arms/RUpperArm.stl scale=0.1 0.1 0.1; visual mesh filename=package://hros5_description/meshes/arms/RUpperArm.dae scale=0.1 0.1 0.1
- link UpperHeadBack: geometry collision mesh filename=package://hros5_description/meshes/head/UpperHeadBack.stl scale=0.1 0.1 0.1; visual mesh filename=package://hros5_description/meshes/head/UpperHeadBack.dae scale=0.1 0.1 0.1
- link UpperHeadBase: geometry collision mesh filename=package://hros5_description/meshes/head/UpperHeadBase.stl scale=0.1 0.1 0.1; visual mesh filename=package://hros5_description/meshes/head/UpperHeadBase.dae scale=0.1 0.1 0.1
- link UpperHeadMotor: geometry collision mesh filename=package://hros5_description/meshes/head/UpperHeadMotor.stl scale=0.1 0.1 0.1; visual mesh filename=package://hros5_description/meshes/head/UpperHeadMotor.dae scale=0.1 0.1 0.1
- link torso: geometry collision mesh filename=package://hros5_description/meshes/torso/torso.stl scale=0.1 0.1 0.1; visual mesh filename=package://hros5_description/meshes/torso/torso.dae scale=0.1 0.1 0.1
Joints:
- added joint LForearmJoint: type fixed, parent LLowerArm, child LForearm, origin xyz=0 0 -0.075 rpy=-1.5708 3.1416 0
- added joint LGrip: type revolute, parent LHand, child LGripper, origin xyz=0.021 0.008 -0.0205 rpy=-1.5708 -1.5708 1.5708, axis 1 0 0, limit lower=-1.0 upper=0.5 effort=1.0 velocity=1.0
- added joint LWrist: type revolute, parent LForearm, child LHand, origin xyz=0 -0.0205 0 rpy=-3.0949 0 -1.5708, axis 1 0 0, limit lower=-3.14 upper=3.14 effort=1.0 velocity=1.0
- added joint RForearmJoint: type fixed, parent RLowerArm, child RForearm, origin xyz=0 0 -0.075 rpy=-1.5708 3.1416 0
- added joint RGrip: type revolute, parent RHand, child RGripper, origin xyz=0.021 0.008 -0.0205 rpy=-1.5708 -1.5708 1.5708, axis 1 0 0, limit lower=-1.0 upper=0.5 effort=1.0 velocity=1.0
- added joint RWrist: type revolute, parent RForearm, child RHand, origin xyz=0 -0.0205 0 rpy=-3.0949 0 -1.5708, axis 1 0 0, limit lower=-3.14 upper=3.14 effort=1.0 velocity=1.0

File: src/hros5_description/urdf/hros5_control.xacro (robot description, xacro)
@@ -133,4 +133,36 @@
       <plugin>dynamixel_hardware_interface/DynamixelHardware</plugin>
     </hardware>
+	  <joint name="HeadYaw">
+		<command_interface name="position"/>
+		<state_interface name="position"/>
+	  </joint>
+	  <joint name="HeadPitch">
+		<command_interface name="position"/>
+		<state_interface name="position"/>
+	  </joint>
+	  <joint name="LShoulderPitch">
+		<command_interface name="position"/>
+		<state_interface name="position"/>
+	  </joint>
+	  <joint name="LShoulderRoll">
+		<command_interface name="position"/>
+		<state_interface name="position"/>
+	  </joint>
+	  <joint name="LElbowPitch">
+		<command_interface name="position"/>
+		<state_interface name="position"/>
+	  </joint>
+	  <joint name="RShoulderPitch">
+		<command_interface name="position"/>
+		<state_interface name="position"/>
+	  </joint>
+	  <joint name="RShoulderRoll">
+		<command_interface name="position"/>
+		<state_interface name="position"/>
+	  </joint>
+	  <joint name="RElbowPitch">
+		<command_interface name="position"/>
+		<state_interface name="position"/>
+	  </joint>
 	  <joint name="LHipYaw">
 		<command_interface name="position"/>
@@ -180,4 +212,24 @@
 		<command_interface name="position"/>
 		<state_interface name="position"/>
+	  </joint>
+	  <joint name="LWrist">
+		<command_interface name="position"/>
+		<state_interface name="position"/>
+		<state_interface name="velocity"/>
+	  </joint>
+	  <joint name="LGrip">
+		<command_interface name="position"/>
+		<state_interface name="position"/>
+		<state_interface name="velocity"/>
+	  </joint>
+	  <joint name="RWrist">
+		<command_interface name="position"/>
+		<state_interface name="position"/>
+		<state_interface name="velocity"/>
+	  </joint>
+	  <joint name="RGrip">
+		<command_interface name="position"/>
+		<state_interface name="position"/>
+		<state_interface name="velocity"/>
 	  </joint>
 	</ros2_control>

File: src/hros5_description/urdf/hros5_gazebo.xacro (robot description, xacro)
@@ -1,12 +1,4 @@
 <?xml version="1.0"?>
 <robot xmlns:xacro="http://www.ros.org/wiki/xacro">
-<!-- GAZEBO ROS CONTROL AND IMU PLUGIN -->
-    <gazebo>
-        <plugin filename="libgazebo_ros_control.so" name="gazebo_ros_control">
-            <robotNamespace>/hros5</robotNamespace>
-            <robotSimType>gazebo_ros_control/DefaultRobotHWSim</robotSimType>
-        </plugin>
-    </gazebo>
-<!-- END OF GAZEBO ROS CONTROL PLUGIN -->
 <!-- MIMIC JOINTS  -->
 	<gazebo>
