Commit message: Reorganized Xacro modules into subsystem folders

File: src/hros5_description/urdf/head/head.xacro (robot description, xacro)
@@ -1,59 +1,70 @@
 <?xml version="1.0"?>
-<robot xmlns:xacro="http://ros.org/wiki/xacro">
-  <link name="LowerHead">
-    <visual>
-      <origin xyz="0 0 0" rpy="0 0 0"/>
-      <geometry>
-        <mesh filename="package://hros5_description/meshes/head/LowerHead.stl" scale="0.1 0.1 0.1"/>
-      </geometry>
-    </visual>
-  </link>
-  <joint name="HeadYaw" type="revolute">
-    <parent link="torso"/>
-    <child link="LowerHead"/>
-    <origin xyz="0 0 0.05" rpy="0 0 0"/>
-    <axis xyz="0 0 1"/>
-    <limit lower="-1.57" upper="1.57" effort="1.0" velocity="1.0"/>
-  </joint>
-  <link name="UpperHeadBase">
-    <visual>
-      <origin xyz="0 0 0" rpy="0 0 0"/>
-      <geometry>
-        <mesh filename="package://hros5_description/meshes/head/UpperHeadBase.stl" scale="0.1 0.1 0.1"/>
-      </geometry>
-    </visual>
-  </link>
-  <joint name="HeadPitch" type="revolute">
-    <parent link="LowerHead"/>
-    <child link="UpperHeadBase"/>
-    <origin xyz="0 0 0.04" rpy="0 0 0"/>
-    <axis xyz="0 1 0"/>
-    <limit lower="-0.8" upper="0.8" effort="1.0" velocity="1.0"/>
-  </joint>
-  <link name="UpperHeadMotor">
-    <visual>
-      <origin xyz="0 0 0" rpy="0 0 0"/>
-      <geometry>
-        <mesh filename="package://hros5_description/meshes/head/UpperHeadMotor.stl" scale="0.1 0.1 0.1"/>
-      </geometry>
-    </visual>
-  </link>
-  <joint name="UpperHeadFixed" type="fixed">
-    <parent link="UpperHeadBase"/>
-    <child link="UpperHeadMotor"/>
-    <origin xyz="0 0 0" rpy="0 0 0"/>
-  </joint>
-  <link name="UpperHeadBack">
-    <visual>
-      <origin xyz="0 0 0" rpy="0 0 0"/>
-      <geometry>
-        <mesh filename="package://hros5_description/meshes/head/UpperHeadBack.stl" scale="0.1 0.1 0.1"/>
-      </geometry>
-    </visual>
-  </link>
-  <joint name="UpperBackFixed" type="fixed">
-    <parent link="UpperHeadBase"/>
-    <child link="UpperHeadBack"/>
-    <origin xyz="0 0 -0.01" rpy="0 0 0"/>
-  </joint>
+<robot xmlns:xacro="http://www.ros.org/wiki/xacro">
+	<joint name="HeadYaw" type="revolute">
+		<parent link="torso"/>
+		<child link="LowerHead"/>
+		<origin xyz="0.0035 0 0.1115" rpy="0 0 0"/>
+		<axis xyz="0 0 1"/>
+		<limit lower="-1.22173048" upper="1.22173048" effort="2.5" velocity="5.759586525"/>
+	</joint>
+	<link name="LowerHead">
+		<xacro:visuals_collisions_lower_head/>
+		<inertial> <!-- Dummy values from Darwin OP -->
+			<origin xyz="0.001424 -0.016567 -0.007128" />
+			<mass value="0.024357719"/>
+			<inertia ixx="0.0051411124"  ixy="-0.00057530255"  ixz="-0.000024729049" iyy="0.0081915737" iyz="-0.000019223094" izz="0.0011379812" />
+	    </inertial>
+	</link>
+	<joint name="HeadPitch" type="revolute">
+		<parent link="LowerHead"/>
+		<child link="UpperHeadBase"/>
+		<origin xyz="-0.01 0 0.049" rpy="0 0 0"/>
+		<axis xyz="0 1 0"/>
+		<limit upper="0.4" lower="-0.25" effort="2.5" velocity="5.759586525"/>
+	</joint>
+	<link name="UpperHeadBase">
+		<xacro:visuals_collisions_upper_head_base/>
+		<inertial> <!-- Dummy values from Darwin OP -->
+			<origin xyz="0.000064 -0.018565 -0.007667" />
+			<mass value="0.15804192"/>
+			<inertia ixx="0.1239683"  ixy="0.000078494368"  ixz="0.000007645979" iyy="0.11783781" iyz="0.0012199205" izz="0.1583601" />
+	    </inertial>
+	</link>
+	<joint name="HeadPitchDummy" type="continuous">
+		<parent link="UpperHeadBase"/>
+		<child link="UpperHeadMotor"/>
+		<origin xyz="-0.00225 0 0.046" rpy="0 0 0"/>
+		<axis xyz="0 1 0"/>
+		<mimic joint="HeadPitch" multiplier="-1.0"/>
+	</joint>
+	<link name="UpperHeadMotor">
+		<xacro:visuals_collisions_upper_head_motor/>
+		<inertial> <!-- dummy values for gazebo -->
+			<mass value="0.2e-5" />
+			<origin xyz="0 0 0"/>
+			<inertia ixx="1e-9" ixy="0" ixz="0" iyy="1e-9" iyz="0" izz="1e-9" />
+		</inertial>
+	</link>
+	<joint name="HeadPitchDummy2" type="continuous">
+		<parent link="LowerHead"/>
+		<child link="UpperHeadBack"/>
+		<origin xyz="-0.0525 0 0.021" rpy="0 0 0"/>
+		<axis xyz="0 1 0"/>
+		<mimic joint="HeadPitch" multiplier="0.65"/>
+	</joint>
+	<link name="UpperHeadBack">
+		<xacro:visuals_collisions_upper_head_back/>
+		<inertial> <!-- dummy values for gazebo -->
+			<mass value="0.2e-5" />
+			<origin xyz="0 0 0"/>
+			<inertia ixx="1e-9" ixy="0" ixz="0" iyy="1e-9" iyz="0" izz="1e-9" />
+		</inertial>
+	</link>
+<!-- ROS REP LINKS -->
+	<joint name="gaze_joint" type="fixed">
+		<parent link="UpperHeadBase"/>
+		<child link="gaze"/>
+		<origin xyz="0 0 0" rpy="0 0 0"/>
+	</joint>
+	<link name="gaze"/>
 </robot>

File: src/hros5_description/urdf/hros5.xacro (robot description, xacro)
@@ -3,4 +3,4 @@
 	<xacro:include filename="$(find hros5_description)/urdf/hros5_control.xacro" />
 	<xacro:include filename="$(find hros5_description)/urdf/hros5_gazebo.xacro" />
-	<xacro:include filename="$(find hros5_description)/urdf/modules/robot.xacro" />
+	<xacro:include filename="$(find hros5_description)/urdf/robot/robot.xacro" />
 </robot>

File: src/hros5_description/urdf/robot/robot.xacro (robot description, xacro)
@@ -6,10 +6,10 @@
 	<xacro:property name="scale" value="0.1" />
 	<xacro:include filename="$(arg meshes_xacro_filename)" />
-	<!-- Load xacro modules/parts of the robot -->
-	<xacro:include filename="$(find hros5_description)/urdf/modules/torso.xacro" />
-	<xacro:include filename="$(find hros5_description)/urdf/modules/head.xacro" />
-	<xacro:include filename="$(find hros5_description)/urdf/modules/arms.xacro" />
-	<!-- <xacro:include filename="$(find hros5_description)/urdf/modules/hands.xacro" /> -->
-	<xacro:include filename="$(find hros5_description)/urdf/modules/legs.xacro" />
+	<!-- Load xacro subparts of the robot -->
+	<xacro:include filename="$(find hros5_description)/urdf/torso/torso.xacro" />
+	<xacro:include filename="$(find hros5_description)/urdf/head/head.xacro" />
+	<xacro:include filename="$(find hros5_description)/urdf/arms/arms.xacro" />
+	<!-- <xacro:include filename="$(find hros5_description)/urdf/hands/hands.xacro" /> -->
+	<xacro:include filename="$(find hros5_description)/urdf/legs/legs.xacro" />
 	<!-- <xacro:include filename="$(find hros5_description)/urdf/modules/imu.xacro" />
 	<xacro:include filename="$(find hros5_description)/urdf/modules/cameras.xacro" /> -->

File: src/hros5_description/urdf/torso/torso.xacro (robot description, xacro)
@@ -1,30 +1,18 @@
 <?xml version="1.0"?>
 <robot xmlns:xacro="http://www.ros.org/wiki/xacro">
-  <!-- Dummy root link -->
-  <link name="base_link"/>
-  <joint name="fixed-base" type="fixed">
-    <parent link="base_link"/>
-    <child link="torso"/>
-  </joint>
-  <!-- TORSO -->
-  <link name="torso">
-    <visual>
-      <origin xyz="0 0 0" rpy="0 0 0"/>
-      <geometry>
-        <mesh filename="package://hros5_description/meshes/torso/torso.stl" scale="0.1 0.1 0.1"/>
-      </geometry>
-    </visual>
-    <collision>
-      <origin xyz="0 0 0" rpy="0 0 0"/>
-      <geometry>
-        <mesh filename="package://hros5_description/meshes/torso/torso.stl" scale="0.1 0.1 0.1"/>
-      </geometry>
-    </collision>
-    <inertial>
-      <origin xyz="-0.003053 -0.038651 -0.019268"/>
-      <mass value="0.97559947"/>
-      <inertia ixx="3.1081800"  ixy="-0.25460189"  ixz="2.0318174"
-               iyy="6.3787776"  iyz="0.16417863"  izz="5.3316425"/>
-    </inertial>
-  </link>
+	<!-- DUMMY ROOT LINK -->
+	<link name="base_link"/>
+	<joint name="fixed-base" type="fixed">
+		<parent link="base_link"/>
+		<child link="torso"/>
+	</joint>
+	<!-- TORSO -->
+	<link name="torso">
+		<xacro:visuals_collisions_torso/>
+		<inertial> <!-- Dummy values from Darwin OP -->
+			<origin xyz="-0.003053 -0.038651 -0.019268" />
+			<mass value="0.97559947"/>
+			<inertia ixx="3.1081800"  ixy="-0.25460189"  ixz="2.0318174" iyy="6.3787776" iyz="0.16417863" izz="5.3316425" />
+		</inertial>
+	</link>
 </robot>

Commit message: Gazebo: add full HR-OS5 bringup, sim controllers, and mesh toggle
- New hros5_gazebo.launch.py with gz sim, spawn params, controller spawners, clock bridge, and resource/plugin envs
- Add full sim URDF + controllers config and fix gz ros2_control plugin names
- Add STL visuals xacro for Gazebo and restore DAE visuals for RViz; launch toggle use_dae_meshes
- Update head mimic joints for Gazebo, inertia fix, and world with inline ground/light + GUI camera
- Wire package deps and controller YAML layout

File: src/hros5_description/urdf/head/head.xacro (robot description, xacro)
@@ -10,8 +10,8 @@
 	<link name="LowerHead">
 		<xacro:visuals_collisions_lower_head/>
-		<inertial> <!-- Dummy values from Darwin OP -->
-			<origin xyz="0.001424 -0.016567 -0.007128" />
-			<mass value="0.024357719"/>
-			<inertia ixx="0.0051411124"  ixy="-0.00057530255"  ixz="-0.000024729049" iyy="0.0081915737" iyz="-0.000019223094" izz="0.0011379812" />
+		<inertial> <!-- Simplified to keep inertia positive definite in simulation -->
+			<origin xyz="0 0 0"/>
+			<mass value="0.1"/>
+			<inertia ixx="0.001" ixy="0.0" ixz="0.0" iyy="0.001" iyz="0.0" izz="0.001" />
 	    </inertial>
 	</link>
@@ -31,10 +31,9 @@
 	    </inertial>
 	</link>
-	<joint name="HeadPitchDummy" type="continuous">
+	<!-- Gazebo Harmonic does not support mimic constraints; keep the dummy links fixed to avoid physics errors. -->
+	<joint name="HeadPitchDummy" type="fixed">
 		<parent link="UpperHeadBase"/>
 		<child link="UpperHeadMotor"/>
 		<origin xyz="-0.00225 0 0.046" rpy="0 0 0"/>
-		<axis xyz="0 1 0"/>
-		<mimic joint="HeadPitch" multiplier="-1.0"/>
 	</joint>
 	<link name="UpperHeadMotor">
@@ -46,10 +45,8 @@
 		</inertial>
 	</link>
-	<joint name="HeadPitchDummy2" type="continuous">
+	<joint name="HeadPitchDummy2" type="fixed">
 		<parent link="LowerHead"/>
 		<child link="UpperHeadBack"/>
 		<origin xyz="-0.0525 0 0.021" rpy="0 0 0"/>
-		<axis xyz="0 1 0"/>
-		<mimic joint="HeadPitch" multiplier="0.65"/>
 	</joint>
 	<link name="UpperHeadBack">

File: src/hros5_description/urdf/robot/robot.xacro (robot description, xacro)
@@ -2,10 +2,11 @@
 <robot xmlns:xacro="http://www.ros.org/wiki/xacro">
 <!-- Note: This file is included by hros5.xacro and is not intended as a standalone entry point -->
-  <!-- Argument with fallback -->
-  <xacro:arg name="meshes_xacro_filename" default="$(find hros5_description)/urdf/hros5_visuals_collisions_endoskeleton.xacro"/>
+	<!-- Argument with fallback -->
+	<xacro:arg name="meshes_xacro_filename" default="$(find hros5_description)/urdf/hros5_visuals_collisions_endoskeleton.xacro"/>
+	<xacro:arg name="scale" default="0.1"/>
 	<!-- XACRO PROPERTIES -->
 	<xacro:property name="PI" value="3.14159265359" />
 	<xacro:property name="PI_2" value="1.57079632679" />
-	<xacro:property name="scale" value="0.1" />
+	<xacro:property name="scale" value="$(arg scale)" />
  <!-- Include shared geometry macros -->
 	<xacro:include filename="$(arg meshes_xacro_filename)" />
